Commit message: improved vlm training

File: cliport/environments/assets/stacking/stand.urdf (robot description, URDF)
Before this commit: robot stand.urdf, 3 links, 2 joints
Links:
- link base1: geometry collision box size=.06 .05 .005; visual box size=.06 .05 .005
- link base2: geometry collision box size=.06 .05 .005; visual box size=.06 .05 .005
- link baseLink: geometry collision box size=.06 .05 .005; visual box size=.06 .05 .005
