Commit message: 0630

File: cliport/environments/assets/trash_can/trashcan.urdf (robot description, URDF)
Before this commit: robot trashcan.urdf, 1 links, 0 joints
Links:
- link baseLink: mass 1.0 -> .1; geometry collision mesh filename=trashcan_1.obj scale=0.07 0.07 0.05; visual mesh filename=trashcan_1.obj scale=0.07 0.07 0.05

Commit message: 1006

File: cliport/environments/assets/trash_can/trashcan.urdf (robot description, URDF)
Before this commit: robot trashcan.urdf, 1 links, 0 joints
Links:
- link baseLink: geometry collision mesh filename=trashcan_1.obj scale=0.07 0.07 0.07; visual mesh filename=trashcan_1.obj scale=0.07 0.07 0.07
